File: kicad/CANFD-Transceiver-Breakout-Board-MCP2562FD.kicad_pcb (KiCad board)
At the start: 2 copper layers, 46.7 x 16.7 mm, 15 parts, among them J2 1862042, K1 HEADER_MALE_6X1, U1 MCP2562FD-E_SN

Commit message: edited gitignore
Other:
- board text added: "03/2026"
- board text added: "CAN HIGH"
- board text added: "CAN LOW"
Changed lines of the file:
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@@
 		(tenting front back)
 		(pcbplotparams
-			(layerselection 0x00000000_00000000_55555555_5755f5ff)
+			(layerselection 0x00000000_00000000_5555555f_f755f5ff)
 			(plot_on_all_layers_selection 0x00000000_00000000_00000000_00000000)
 			(disableapertmacros no)
-			(usegerberextensions no)
+			(usegerberextensions yes)
 			(usegerberattributes yes)
 			(usegerberadvancedattributes yes)
@@
 			(outputformat 1)
 			(mirror no)
-			(drillshape 1)
+			(drillshape 0)
 			(scaleselection 1)
-			(outputdirectory "")
+			(outputdirectory "assembly/")
 		)
 	)
@@
 	)
 	(gr_text "MCP2562FD CANFD XCVR BOARD"
-		(at 122.55 99.8 0)
+		(at 123.2154 99.6442 0)
 		(layer "F.SilkS" knockout)
 		(effects
@@
 		)
 	)
+	(gr_text "CAN HIGH"
+		(at 144.907 87.4776 0)
+		(layer "F.SilkS" knockout)
+		(effects
+			(font
+				(size 0.7 0.7)
+				(thickness 0.0875)
+			)
+			(justify left bottom)
+		)
+	)
+	(gr_text "CAN LOW"
+		(at 145.2626 98.4758 0)
+		(layer "F.SilkS" knockout)
+		(effects
+			(font
+				(size 0.7 0.7)
+				(thickness 0.0875)
+			)
+			(justify left bottom)
+		)
+	)
+	(gr_text "03/2026"
+		(at 127.9906 98.7552 0)
+		(layer "B.SilkS" knockout)
+		(effects
+			(font
+				(size 0.7 0.7)
+				(thickness 0.0875)
+			)
+			(justify left bottom mirror)
+		)
+	)
 	(gr_text "Atmadyne"
 		(at 135.5 96.75 0)
@@
 	)
 	(via
-		(at 146.625 99.5)
+		(at 148.971 96.0882)
 		(size 0.6)
 		(drill 0.3)
@@
 	)
 	(via
-		(at 145.6 87.775)
+		(at 144.8816 89.0524)
 		(size 0.6)
 		(drill 0.3)
@@
 	)
 	(via
-		(at 149.725 96.125)
+		(at 148.9456 92.4052)
 		(size 0.6)
 		(drill 0.3)

Commit message: refine
Routing:
- net GND: vias 25 -> 29
Changed lines of the file:
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@@
+	)
+	(via
+		(at 121.2088 89.3064)
+		(size 0.6)
+		(drill 0.3)
+		(layers "F.Cu" "B.Cu")
+		(free yes)
+		(net 1)
 	)
 	(via
@@
 	)
 	(via
+		(at 116.967 91.3638)
+		(size 0.6)
+		(drill 0.3)
+		(layers "F.Cu" "B.Cu")
+		(free yes)
+		(net 1)
+	)
+	(via
 		(at 118.35 92.875)
+		(size 0.6)
+		(drill 0.3)
+		(layers "F.Cu" "B.Cu")
+		(free yes)
+		(net 1)
+	)
+	(via
+		(at 137.6172 92.5068)
 		(size 0.6)
 		(drill 0.3)
@@
 		(size 0.6)
 		(drill 0.3)
+		(layers "F.Cu" "B.Cu")
+		(free yes)
+		(net 1)
+	)
+	(via
+		(at 135.6 92.5)
+		(size 0.6)
+		(drill 0.3)

Commit message: refine
Parts:
- added H1: HOLE_2.2mm, MountingHole:MountingHole_2.2mm_M2_DIN965_Pad_TopBottom, F.Cu at (134.0, 97.8)
- added H3: HOLE_2.2mm, MountingHole:MountingHole_2.2mm_M2_DIN965_Pad_TopBottom, F.Cu at (134.0, 86.8)
Other:
- board text added: "CANFD XCVR BOARD"
- board text added: "MCP2562FD"
- board text removed: "MCP2562FD CANFD XCVR BOARD"
