File: kicad/CANFD-Transceiver-Breakout-Board-MCP2562FD.kicad_pcb (KiCad board)
At the start: 2 copper layers, 46.7 x 16.7 mm, 17 parts, among them J2 1862042, K1 HEADER_MALE_6X1, U1 MCP2562FD-E_SN

Commit message: final revision
Parts:
- added G***: LOGO, LOGO, B.Cu at (126.6, 92.6)
- moved D1 0.46 mm to (117.9, 98.0)
- moved R3 0.46 mm to (114.3, 98.0)
Routing:
- net 3V3: track 19.4 -> 21.1 mm
- net GND: vias 29 -> 31
Changed lines of the file:
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@@
 	(footprint "Resistor_SMD:R_0603_1608Metric_Pad0.98x0.95mm_HandSolder"
 		(layer "F.Cu")
-		(at 114.3 97.536)
+		(at 114.3 98)
 		(descr "Resistor SMD 0603 (1608 Metric), square (rectangular) end terminal, IPC-7351 nominal with elongated pad for handsoldering. (Body size source: IPC-SM-782 page 72, https://www.pcb-3d.com/wordpress/wp-content/uploads/ipc-sm-782a_amendment_1_and_2.pdf), generated with kicad-footprint-generator")
 		(tags "resistor handsolder")
@@
 	(footprint "LED_SMD:LED_0603_1608Metric_Pad1.05x0.95mm_HandSolder"
 		(layer "F.Cu")
-		(at 117.9208 97.536 180)
+		(at 117.9208 98 180)
 		(descr "LED SMD 0603 (1608 Metric), square (rectangular) end terminal, IPC-7351 nominal, (Body size source: http://www.tortai-tech.com/upload/download/2011102023233369053.pdf), generated with kicad-footprint-generator")
 		(tags "LED handsolder")
@@
 		)
 	)
+	(footprint "LOGO"
+		(layer "B.Cu")
+		(at 126.6 92.6 180)
+		(property "Reference" "G***"
+			(at 0 0 0)
+			(layer "B.SilkS")
+			(hide yes)
+			(effects
+				(font
+					(size 1.5 1.5)
+					(thickness 0.3)
+				)
+				(justify mirror)
+			)
+		)
+		(property "Value" "LOGO"
+			(at 0.75 0 0)
+			(layer "B.SilkS")
+			(hide yes)
+			(effects
+				(font
+					(size 1.5 1.5)
+					(thickness 0.3)
+				)
+				(justify mirror)
+			)
+		)
+		(property "Datasheet" ""
+			(at 0 0 0)
+			(layer "B.Fab")
+			(hide yes)
+			(effects
+				(font
+					(size 1.27 1.27)
+					(thickness 0.15)
+				)
+				(justify mirror)
+			)
+		)
+		(property "Description" ""
+			(at 0 0 0)
+			(layer "B.Fab")
+			(hide yes)
+			(effects
+				(font
+					(size 1.27 1.27)
+					(thickness 0.15)
+				)
+				(justify mirror)
+			)
+		)
+		(attr board_only exclude_from_pos_files exclude_from_bom)
+		(fp_poly
+			(pts
+				(xy -0.729893 3.745247) (xy 2.408903 3.736258) (xy 2.585148 3.664077) (xy 2.875383 3.511256) (xy 3.131689 3.307997)
+				(xy 3.346672 3.062685) (xy 3.512941 2.783706) (xy 3.620526 2.489477) (xy 3.629275 2.448946) (xy 3.63697 2.396015)
+				(xy 3.643675 2.326583) (xy 3.649456 2.236552) (xy 3.654378 2.121822) (xy 3.658505 1.978293) (xy 3.661902 1.801865)
+				(xy 3.664635 1.588439) (xy 3.666768 1.333915) (xy 3.668366 1.034193) (xy 3.669494 0.685174) (xy 3.670218 0.282759)
+				(xy 3.670601 -0.177153) (xy 3.67071 -0.678757) (xy 3.67071 -3.654322) (xy 0.64729 -3.651576) (xy 0.08308 -3.650804)
+				(xy -0.418307 -3.649549) (xy -0.859596 -3.647775) (xy -1.243509 -3.645446) (xy -1.572771 -3.642527)
+				(xy -1.850106 -3.638982) (xy -2.078238 -3.634775) (xy -2.259891 -3.629871) (xy -2.397789 -3.624235)
+				(xy -2.494655 -3.61783) (xy -2.553214 -3.610621) (xy -2.557982 -3.60966) (xy -2.844159 -3.515503)
+				(xy -3.110608 -3.36449) (xy -3.349068 -3.164306) (xy -3.551277 -2.922634) (xy -3.708973 -2.647157)
+				(xy -3.776155 -2.476815) (xy -3.79308 -2.42361) (xy -3.807188 -2.370472) (xy -3.818796 -2.310959)
+				(xy -3.828216 -2.238631) (xy -3.835765 -2.147044) (xy -3.841757 -2.029757) (xy -3.846507 -1.880326)
+				(xy -3.850329 -1.692311) (xy -3.853539 -1.459269) (xy -3.85645 -1.174758) (xy -3.859379 -0.832336)
+				(xy -3.859949 -0.762) (xy -3.861733 -0.540774) (xy -2.494206 -0.540774) (xy -2.484329 -1.307597)
+				(xy -2.480835 -1.552695) (xy -2.476959 -1.740829) (xy -2.47193 -1.880586) (xy -2.464978 -1.980548)
+				(xy -2.455331 -2.049302) (xy -2.442218 -2.09543) (xy -2.424867 -2.127518) (xy -2.408903 -2.147207)
+				(xy -2.338021 -2.210494) (xy -2.277807 -2.246823) (xy -2.234686 -2.251365) (xy -2.131516 -2.255724)
+				(xy -1.973797 -2.259832) (xy -1.767026 -2.263621) (xy -1.516703 -2.267022) (xy -1.228328 -2.269967)
+				(xy -0.907399 -2.272386) (xy -0.559415 -2.274212) (xy -0.189876 -2.275376) (xy 0.040968 -2.275729)
+				(xy 2.294193 -2.277806) (xy 2.294193 -1.40929) (xy 2.294193 -0.540774) (xy -0.100006 -0.540774)
+				(xy -2.494206 -0.540774) (xy -3.861733 -0.540774) (xy -3.87204 0.737419) (xy -0.788923 0.737419)
+				(xy 2.294193 0.737419) (xy 2.294193 1.456624) (xy 2.294013 1.691451) (xy 2.29288 1.869856) (xy 2.289904 2.000965)
+				(xy 2.284195 2.093902) (xy 2.274864 2.157796) (xy 2.26102 2.20177) (xy 2.241774 2.234952) (xy 2.216236 2.266467)
+				(xy 2.215102 2.267785) (xy 2.136011 2.359742) (xy -0.857478 2.376129) (xy -3.850968 2.392516) (xy -3.859829 3.073376)
+				(xy -3.86869 3.754236)
+			)
+			(stroke
+				(width 0)
+				(type solid)
+			)
+			(fill yes)
+			(layer "B.SilkS")
+		)
+		(embedded_fonts no)
+	)
 	(gr_line
 		(start 104.45 83.852)
@@
 		)
 	)
-	(gr_text "03/2026"
-		(at 121.0056 88.5952 0)
+	(gr_text "Atmadyne"
+		(at 121.2 91.2 0)
 		(layer "B.SilkS" knockout)
 		(effects
@@
 		)
 	)
-	(gr_text "Atmadyne"
-		(at 125.0188 86.0552 0)
+	(gr_text "Jonathan Lin"
+		(at 121.2 93.2 0)
 		(layer "B.SilkS" knockout)
 		(effects
@@
 		)
 	)
-	(gr_text "Jonathan Lin"
-		(at 128.515 88.59 0)
+	(gr_text "03/2026"
+		(at 121.2 95 0)
 		(layer "B.SilkS" knockout)
 		(effects
@@
 	)
 	(via
+		(at 144.2 99.4)
+		(size 0.6)
+		(drill 0.3)
+		(layers "F.Cu" "B.Cu")
+		(free yes)
+		(net 1)
+	)
+	(via
 		(at 116.967 91.3638)
 		(size 0.6)
@@
 	)
 	(via
-		(at 118.35 95.175)
+		(at 119.4 95)
 		(size 0.6)
 		(drill 0.3)
@@
 	)
 	(via
+		(at 138 99.4)
+		(size 0.6)
+		(drill 0.3)
+		(layers "F.Cu" "B.Cu")
+		(free yes)
+		(net 1)
+	)
+	(via
 		(at 131 85.225)
 		(size 0.6)
@@
 	)
 	(via
-		(at 111.9 95)
+		(at 112 94.8)
 		(size 0.6)
 		(drill 0.3)
@@
 		(start 121.2088 95.7845)
 		(end 121.2088 93.9138)
-		(width 0.2)
+		(width 0.6)
 		(layer "F.Cu")
 		(net 3)
@@
 	(segment
 		(start 109 96.04)
-		(end 120.9533 96.04)
-		(width 0.5)
+		(end 109.24 95.8)
+		(width 0.6)
 		(layer "F.Cu")
 		(net 3)
 	)
 	(segment
-		(start 112.296 96.04)
-		(end 109 96.04)
-		(width 0.2)
+		(start 113.3875 96.8875)
+		(end 113.3875 96.7875)
+		(width 0.6)
 		(layer "F.Cu")
 		(net 3)
 	)
 	(segment
-		(start 113.3875 97.1315)
-		(end 112.296 96.04)
-		(width 0.5)
+		(start 109.24 95.8)
+		(end 121.1933 95.8)
+		(width 0.6)
 		(layer "F.Cu")
 		(net 3)
 	)
 	(segment
-		(start 113.3875 97.536)
-		(end 113.3875 97.1315)
-		(width 0.5)
+		(start 113.3875 96.7875)
+		(end 112.4 95.8)
+		(width 0.6)
+		(layer "F.Cu")
+		(net 3)
+	)
+	(segment
+		(start 112.4 95.8)
+		(end 109.24 95.8)
+		(width 0.6)
+		(layer "F.Cu")
+		(net 3)
+	)
+	(segment
+		(start 113.3875 96.8875)
+		(end 113.3875 98)
+		(width 0.6)
+		(layer "F.Cu")
+		(net 3)
+	)
+	(segment
+		(start 121.1933 95.8)
+		(end 121.2088 95.7845)
+		(width 0.6)
 		(layer "F.Cu")
 		(net 3)
@@
 		(start 121.2088 93.9138)
 		(end 121.2 93.905)
+		(width 0.6)
+		(layer "F.Cu")
+		(net 3)
+	)
+	(segment
+		(start 113.3875 98)
+		(end 113.3875 97.536)
 		(width 0.2)
 		(layer "F.Cu")
@@
 	)
 	(segment
-		(start 120.9533 96.04)
-		(end 121.2088 95.7845)
-		(width 0.5)
+		(start 113.3875 97.536)
+		(end 113.3875 96.8875)
+		(width 0.6)
 		(layer "F.Cu")
 		(net 3)
 	)
 	(segment
-		(start 115.2125 97.536)
-		(end 117.0458 97.536)
+		(start 115.2125 98)
+		(end 117.0458 98)
 		(width 0.7)
 		(layer "F.Cu")
